Commit message: Update README.md

File: ros/catkin_ws/src/husky_description/urdf/husky_OS1-64_arch.urdf.xacro (robot description, xacro)
@@ -314,5 +314,5 @@
          <box size="0.762 0.610 0.267" />
         </geometry>
-        <material name="dark_grey"/>
+        <material name="red"/>
      </visual>
      <collision>

Commit message: Add os_imu location in robot urdf

File: ros/catkin_ws/src/husky_description/urdf/husky_OS1-64_arch.urdf.xacro (robot description, xacro)
@@ -379,4 +379,13 @@
  <!--     <parent link="base_link"/>    -->
       <child link="os_sensor"/>
-    </joint>
+   </joint>
+ <!--
+      Ouster Link for imu (separate from ouster lidar data
+  -->
+   <link name="os_imu"/>
+   <joint name="os_imu_joint" type="fixed">
+     <parent link="OS1_sensor_arch_mount_link"/>
+     <child link="os_imu" />
+     <origin xyz="0.006253 -0.011775 0.007645" rpy="0 0 0" />
+   </joint>
 </robot>
